Commit message: Use iCub 2.5 by default

File: icub_description/urdf/icub_2_5.urdf (robot description, URDF)
Before this commit: robot ICUB_2-5_BB_SIM_MODEL, 107 links, 106 joints
Links:
- link chest: geometry collision mesh filename=package://icub_description/meshes/icub2_5/visual/chest.dae scale=0.001 0.001 0.001; visual mesh filename=package://icub_description/meshes/icub2_5/visual/chest.dae scale=0.001 0.001 0.001
- link head: geometry collision mesh filename=package://icub_description/meshes/icub2_5/visual/head.dae scale=0.001 0.001 0.001; visual mesh filename=package://icub_description/meshes/icub2_5/visual/head.dae scale=0.001 0.001 0.001
- link l_ankle_1: geometry collision mesh filename=package://icub_description/meshes/icub2_5/visual/l_ankle_1.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 scale=0.001 0.001 0.001; visual mesh filename=package://icub_description/meshes/icub2_5/visual/l_ankle_1.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 scale=0.001 0.001 0.001
- link l_ankle_2: geometry collision mesh filename=package://icub_description/meshes/icub2_5/visual/l_ankle_2.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 scale=0.001 0.001 0.001; visual mesh filename=package://icub_description/meshes/icub2_5/visual/l_ankle_2.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 scale=0.001 0.001 0.001
- link l_elbow_1: geometry collision mesh filename=package://icub_description/meshes/icub2_5/visual/l_elbow_1.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 scale=0.001 0.001 0.001; visual mesh filename=package://icub_description/meshes/icub2_5/visual/l_elbow_1.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 scale=0.001 0.001 0.001
- link l_foot: geometry collision mesh filename=package://icub_description/meshes/icub2_5/visual/l_foot.dae scale=0.001 0.001 0.001; visual mesh filename=package://icub_description/meshes/icub2_5/visual/l_foot.dae scale=0.001 0.001 0.001
- link l_forearm: geometry collision mesh filename=package://icub_description/meshes/visual/icub_l_forearm.dae scale=0.001 0.001 0.001; visual mesh filename=package://icub_description/meshes/visual/icub_l_forearm.dae scale=0.001 0.001 0.001
- link l_hand: geometry collision mesh filename=package://icub_description/meshes/visual/icub_l_hand.dae scale=0.001 0.001 0.001; visual mesh filename=package://icub_description/meshes/visual/icub_l_hand.dae scale=0.001 0.001 0.001
- link l_hip_1: geometry collision mesh filename=package://icub_description/meshes/icub2_5/visual/l_hip_1.dae scale=0.001 0.001 0.001; visual mesh filename=package://icub_description/meshes/icub2_5/visual/l_hip_1.dae scale=0.001 0.001 0.001
- link l_hip_2: geometry collision mesh filename=package://icub_description/meshes/icub2_5/visual/l_hip_2.dae scale=0.001 0.001 0.001; visual mesh filename=package://icub_description/meshes/icub2_5/visual/l_hip_2.dae scale=0.001 0.001 0.001
- link l_lower_leg: geometry collision mesh filename=package://icub_description/meshes/icub2_5/visual/l_lower_le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 scale=0.001 0.001 0.001; visual mesh filename=package://icub_description/meshes/icub2_5/visual/l_lower_le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 scale=0.001 0.001 0.001
- link l_shoulder_1: geometry collision mesh filename=package://icub_description/meshes/icub2_5/visual/l_shoulder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 scale=0.001 0.001 0.001; visual mesh filename=package://icub_description/meshes/icub2_5/visual/l_shoulder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 scale=0.001 0.001 0.001
- link l_shoulder_2: geometry collision mesh filename=package://icub_description/meshes/icub2_5/visual/l_shoulder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 scale=0.001 0.001 0.001; visual mesh filename=package://icub_description/meshes/icub2_5/visual/l_shoulder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 scale=0.001 0.001 0.001
- link l_shoulder_3: geometry collision mesh filename=package://icub_description/meshes/icub2_5/visual/l_shoulder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 scale=0.001 0.001 0.001; visual mesh filename=package://icub_description/meshes/icub2_5/visual/l_shoulder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 scale=0.001 0.001 0.001
- link l_upper_arm: geometry collision mesh filename=package://icub_description/meshes/icub2_5/visual/l_upper_ar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 scale=0.001 0.001 0.001; visual mesh filename=package://icub_description/meshes/icub2_5/visual/l_upper_ar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 scale=0.001 0.001 0.001
- link l_upper_leg: geometry collision mesh filename=package://icub_description/meshes/icub2_5/visual/l_upper_le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 scale=0.001 0.001 0.001; visual mesh filename=package://icub_description/meshes/icub2_5/visual/l_upper_le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 scale=0.001 0.001 0.001
- link l_wrist_1: geometry 
- link neck_1: geometry collision mesh filename=package://icub_description/meshes/icub2_5/visual/neck_1.dae scale=0.001 0.001 0.001; visual mesh filename=package://icub_description/meshes/icub2_5/visual/neck_1.dae scale=0.001 0.001 0.001
- link neck_2: geometry collision mesh filename=package://icub_description/meshes/icub2_5/visual/neck_2.dae scale=0.001 0.001 0.001; visual mesh filename=package://icub_description/meshes/icub2_5/visual/neck_2.dae scale=0.001 0.001 0.001
- link r_ankle_1: geometry collision mesh filename=package://icub_description/meshes/icub2_5/visual/r_ankle_1.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 scale=0.001 0.001 0.001; visual mesh filename=package://icub_description/meshes/icub2_5/visual/r_ankle_1.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 scale=0.001 0.001 0.001
- link r_ankle_2: geometry collision mesh filename=package://icub_description/meshes/icub2_5/visual/r_ankle_2.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 scale=0.001 0.001 0.001; visual mesh filename=package://icub_description/meshes/icub2_5/visual/r_ankle_2.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 scale=0.001 0.001 0.001
- link r_elbow_1: geometry collision mesh filename=package://icub_description/meshes/icub2_5/visual/r_elbow_1.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 scale=0.001 0.001 0.001; visual mesh filename=package://icub_description/meshes/icub2_5/visual/r_elbow_1.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 scale=0.001 0.001 0.001
- link r_foot: geometry collision mesh filename=package://icub_description/meshes/icub2_5/visual/r_foot.dae scale=0.001 0.001 0.001; visual mesh filename=package://icub_description/meshes/icub2_5/visual/r_foot.dae scale=0.001 0.001 0.001
- link r_forearm: geometry collision mesh filename=package://icub_description/meshes/visual/icub_r_forearm.dae scale=0.001 0.001 0.001; visual mesh filename=package://icub_description/meshes/visual/icub_r_forearm.dae scale=0.001 0.001 0.001
- link r_hand: geometry collision mesh filename=package://icub_description/meshes/visual/icub_r_hand.dae scale=0.001 0.001 0.001; visual mesh filename=package://icub_description/meshes/visual/icub_r_hand.dae scale=0.001 0.001 0.001
- link r_hip_1: geometry collision mesh filename=package://icub_description/meshes/icub2_5/visual/r_hip_1.dae scale=0.001 0.001 0.001; visual mesh filename=package://icub_description/meshes/icub2_5/visual/r_hip_1.dae scale=0.001 0.001 0.001
- link r_hip_2: geometry collision mesh filename=package://icub_description/meshes/icub2_5/visual/r_hip_2.dae scale=0.001 0.001 0.001; visual mesh filename=package://icub_description/meshes/icub2_5/visual/r_hip_2.dae scale=0.001 0.001 0.001
- link r_lower_leg: geometry collision mesh filename=package://icub_description/meshes/icub2_5/visual/r_lower_le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 scale=0.001 0.001 0.001; visual mesh filename=package://icub_description/meshes/icub2_5/visual/r_lower_le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 scale=0.001 0.001 0.001
- link r_shoulder_1: geometry collision mesh filename=package://icub_description/meshes/icub2_5/visual/r_shoulder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 scale=0.001 0.001 0.001; visual mesh filename=package://icub_description/meshes/icub2_5/visual/r_shoulder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 scale=0.001 0.001 0.001
- link r_shoulder_2: geometry collision mesh filename=package://icub_description/meshes/icub2_5/visual/r_shoulder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 scale=0.001 0.001 0.001; visual mesh filename=package://icub_description/meshes/icub2_5/visual/r_shoulder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 scale=0.001 0.001 0.001
- link r_shoulder_3: geometry collision mesh filename=package://icub_description/meshes/icub2_5/visual/r_shoulder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 scale=0.001 0.001 0.001; visual mesh filename=package://icub_description/meshes/icub2_5/visual/r_shoulder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 scale=0.001 0.001 0.001
- link r_upper_arm: geometry collision mesh filename=package://icub_description/meshes/icub2_5/visual/r_upper_ar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 scale=0.001 0.001 0.001; visual mesh filename=package://icub_description/meshes/icub2_5/visual/r_upper_ar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 scale=0.001 0.001 0.001
- link r_upper_leg: geometry collision mesh filename=package://icub_description/meshes/icub2_5/visual/r_upper_le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 scale=0.001 0.001 0.001; visual mesh filename=package://icub_description/meshes/icub2_5/visual/r_upper_le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 scale=0.001 0.001 0.001
- link r_wrist_1: geometry 
- link root_link: geometry collision box size=0.01 0.01 0.01; visual box size=0.01 0.01 0.01
- link torso_1: geometry collision mesh filename=package://icub_description/meshes/icub2_5/visual/torso_1.dae scale=0.001 0.001 0.001; visual mesh filename=package://icub_description/meshes/icub2_5/visual/torso_1.dae scale=0.001 0.001 0.001

Commit message: Use flipped mesh

File: icub_description/urdf/icub_2_5.urdf (robot description, URDF)
Before this commit: robot ICUB_2-5_BB_SIM_MODEL, 107 links, 106 joints
Links:
- link chest: geometry collision mesh filename=package://icub_description/meshes/icub2_5/visual/bb_chest.d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 scale=0.001 0.001 0.001; visual mesh filename=package://icub_description/meshes/icub2_5/visual/bb_chest.d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 scale=0.001 0.001 0.001

Commit message: Fix root link name, this adds diapers

File: icub_description/urdf/icub_2_5.urdf (robot description, URDF)
Before this commit: robot ICUB_2-5_BB_SIM_MODEL, 107 links, 106 joints
Links:
- link root_link: geometry collision mesh filename=package://icub_description/meshes/icub2_5/visual/root.dae scale=0.001 0.001 0.001; visual mesh filename=package://icub_description/meshes/icub2_5/visual/root.dae scale=0.001 0.001 0.001
